File: yearling-electronics-ChristeenZ/EPS V0/AltRegs.kicad_sch (KiCad schematic)
At the start: 2 parts

Commit message: Add files via upload
im so sorry for the million V0 backup files XD this has the 'V1" schem with new solar and ADC ckt
Parts:
- C1: value (none) -> 22uF
- U?: value (none) -> LT1963AxQ-3.3; footprint (none) -> Package_TO_SOT_SMD:TO-263-5_TabPin3
Changed lines of the file:
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@@
       (effects (font (size 1.27 1.27)) hide)
     )
-    (property "Value" "" (id 1) (at 62.23 62.8634 0))
+    (property "Value" "GND" (id 1) (at 62.23 62.8634 0))
     (property "Footprint" "" (id 2) (at 62.23 58.42 0)
       (effects (font (size 1.27 1.27)) hide)
@@
     (in_bom yes) (on_board yes) (fields_autoplaced)
     (property "Reference" "U?" (id 0) (at 52.07 36.9402 0))
-    (property "Value" "" (id 1) (at 52.07 39.4771 0))
-    (property "Footprint" "" (id 2) (at 52.07 57.15 0)
+    (property "Value" "LT1963AxQ-3.3" (id 1) (at 52.07 39.4771 0))
+    (property "Footprint" "Package_TO_SOT_SMD:TO-263-5_TabPin3" (id 2) (at 52.07 57.15 0)
       (effects (font (size 1.27 1.27)) hide)
     )
@@
       (effects (font (size 1.27 1.27)) (justify left))
     )
-    (property "Value" "" (id 1) (at 76.581 51.2322 0)
+    (property "Value" "22uF" (id 1) (at 76.581 51.2322 0)
       (effects (font (size 1.27 1.27)) (justify left))
     )
