File: yearling-electronics-ChristeenZ/EPS V0/Battery.kicad_sch (KiCad schematic)
At the start: 8 parts, among them U2 1043, U3 1043, U4 1043, U6 BQ29702

Commit message: Add files via upload
im so sorry for the million V0 backup files XD this has the 'V1" schem with new solar and ADC ckt
Parts:
- U1: value (none) -> 1043; footprint (none) -> 1043_KEY
- U5: value (none) -> BQ29702; footprint (none) -> Package_SON:WSON-6_1.5x1.5mm_P0.5mm
- U6: value (none) -> IRF7503TRPBF; footprint (none) -> IRF7503TRPBF_INF
Changed lines of the file:
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@@
       (effects (font (size 1.524 1.524)))
     )
-    (property "Value" "" (id 1) (at 80.01 42.0258 0)
+    (property "Value" "1043" (id 1) (at 80.01 42.0258 0)
       (effects (font (size 1.524 1.524)))
     )
-    (property "Footprint" "" (id 2) (at 80.01 42.164 0)
+    (property "Footprint" "1043_KEY" (id 2) (at 80.01 42.164 0)
       (effects (font (size 1.524 1.524)) hide)
     )
@@
       (effects (font (size 1.524 1.524)))
     )
-    (property "Value" "" (id 1) (at 143.51 111.8758 0)
+    (property "Value" "IRF7503TRPBF" (id 1) (at 143.51 111.8758 0)
       (effects (font (size 1.524 1.524)))
     )
-    (property "Footprint" "" (id 2) (at 143.51 112.014 0)
+    (property "Footprint" "IRF7503TRPBF_INF" (id 2) (at 143.51 112.014 0)
       (effects (font (size 1.524 1.524)) hide)
     )
@@
     (in_bom yes) (on_board yes) (fields_autoplaced)
     (property "Reference" "U5" (id 0) (at 130.81 81.3902 0))
-    (property "Value" "" (id 1) (at 130.81 83.9271 0))
-    (property "Footprint" "" (id 2) (at 130.81 81.28 0)
+    (property "Value" "BQ29702" (id 1) (at 130.81 83.9271 0))
+    (property "Footprint" "Package_SON:WSON-6_1.5x1.5mm_P0.5mm" (id 2) (at 130.81 81.28 0)
       (effects (font (size 1.27 1.27)) hide)
     )
