File: yearling-electronics-ChristeenZ/EPS V0/EPS V0.kicad_sch (KiCad schematic)
At the start: 235 parts

Commit message: Add files via upload
im so sorry for the million V0 backup files XD this has the 'V1" schem with new solar and ADC ckt
Parts:
- removed C? (x2): 10u, symbol Device:C
- removed C? (x2): 22n, symbol Device:C
- removed C?: 2.2u, symbol Device:C
- removed C?: C, symbol Device:C
- removed C?: 4.7u, symbol Device:C
- removed C?: 22u, symbol Device:C
- removed C? (x2): 1uF, Capacitor_SMD:C_0402_1005Metric, symbol Device:C_Small
- removed C?: 47n, symbol Device:C
- removed C?: 1u, symbol Device:C
- removed D?: LED, symbol Device:LED
- removed IC?: LTC4121, QFN50P300X300X80-17N-D, symbol LTC4121:LTC4121
- removed IC?: BQ25883RGER, QFN50P400X400X100-25N-D, symbol BQ25883RGER:BQ25883RGER
- removed J?: Conn_01x06, symbol Connector_Generic:Conn_01x06
- removed L?: L, symbol Device:L
- removed L?: 1u, symbol Device:L
- removed R?: 100k, symbol Device:R_US
- removed R?: 464k, symbol Device:R_US
- removed R? (x2): 10k, symbol Device:R_US
- removed R?: 845k, symbol Device:R_US
- removed R?: 121k, symbol Device:R_US
- removed R?: 107k, symbol Device:R_US
- removed R?: 5.23k, symbol Device:R_US
- removed R?: 3.16k, symbol Device:R_US
- removed R?: 3.01k, symbol Device:R_US
- removed R?: 787k, symbol Device:R_US
- removed R?: 30.1k, symbol Device:R_US
- removed R?: 2.1M, symbol Device:R_US
- removed U?: XC6206PxxxMR-Regulator_Linear, Package_TO_SOT_SMD:SOT-23, symbol kicad-keyboard-parts:XC6206PxxxMR-Regulator_Linear
- added C, C? (x26): (no value), symbol Device:C
- added C? (x9): 10u, symbol Device:C
- added C?: C, symbol Device:C
- added C?: 0.1u, symbol Device:C
- added D?: (no value), symbol Diode:BAT42
- added D?: (no value), symbol Device:D
- added IC?: (no value), symbol MCP6V02-E_MD:MCP6V02-E_MD
- added IC?: (no value), symbol INA180B2IDBVT:INA180B2IDBVT
- added IC?: MCP1790T-5002E_DB, SOT230P700X180-4N, symbol MCP1790T-5002E_DB:MCP1790T-5002E_DB
- added IC?: (no value), symbol PIC16F1503-I_P:PIC16F1503-I_P
- added IC?: (no value), symbol MCP14628-E_SN:MCP14628-E_SN
- added J? (x3): (no value), symbol Connector_Generic:Conn_01x02
- added J?: (no value), symbol Connector_Generic:Conn_01x06
- added L? (x2): (no value), symbol Device:L_Ferrite
- added R? (x25): (no value), symbol Device:R_US
- added R? (x3): R_US, symbol Device:R_US
- added SW?: SW_MEC_5E, symbol Switch:SW_MEC_5E
- added SW? (x2): SW_SPST, symbol Switch:SW_SPST
- added SW?: (no value), symbol Switch:SW_SPST
- added TH?: (no value), symbol Device:Thermistor_US
- added U? (x2): (no value), symbol SI4154DY-T1-GE3:SI4154DY-T1-GE3
- added U?: (no value), symbol ADS1119IPW:ADS1119IPW
- C? (x5): value C -> (none)
- L?: value L -> (none)
Connections:
- net DisableCharge1 is gone; now on net VCHRG: IC?.4 (GPIO2)
- net DisableCharge2 is gone; now on net WDT_WDI: IC?.9 (GPIO7)
- net +3V3: now also IC?.40 (GPIO28/ADC2), IC?.41 (GPIO29/ADC3), C?.1, C?.1, C?.1, C?.2, IC?.5 (VS), R?.1, R?.1, R?.2, R?.2, R?.2, R?.2, U?.12 (AVDD), U?.13 (DVDD), U?.9 (REFP)
- net +5V: now also C?.1, C?.1, C?.1, C?.1, C?.1, C?.1, C?.1, IC?.1 (VDD), IC?.3 (VOUT), J?.1 (Pin_1), J?.2 (Pin_2), L?.2, R?.1, R?.1
- net ALRT1_1: now also IC?.36 (GPIO24); no longer IC?.17 (GPIO14)
- net ALRT1_2: now also IC?.37 (GPIO25); no longer IC?.18 (GPIO15)
- net CH_STAT1: no longer IC?.2 (GPIO0)
- net CH_STAT2: no longer IC?.7 (GPIO5)
- net ChargeDisable1: no longer IC?.5 (GPIO3)
- net ChargeDisable2: no longer IC?.11 (GPIO8)
- net DISCH_STAT1: no longer IC?.3 (GPIO1)
- net DISCH_STAT2: no longer IC?.8 (GPIO6)
- net GND: now also C.2, C?.2, C?.2, C?.2, C?.2, C?.2, C?.2, C?.2, C?.2, C?.2, C?.2, C?.2, C?.2, C?.2, C?.2, C?.2, C?.2, C?.2, C?.2, C?.2, D?.1 (K), IC?.14 (VSS), IC?.2 (GND_(TAB)_1), IC?.4 (GND), IC?.4 (GND_(TAB)_2), IC?.4 (VSS), IC?.5 (VINB+), IC?.7 (FCCM), IC?.9 (EP), J?.2 (Pin_2), J?.3 (Pin_3), L?.2, R?.1, R?.1, R?.2, R?.2, R?.2, SW?.1, SW?.3 (K), U?.1 (S), U?.2 (S), U?.3 (S)
- net SCL: now also IC?.10 (RC0)
- net SCL_I2C_1: now also IC?.30 (GPIO19); no longer IC?.12 (GPIO9)
- net SCL_I2C_2: now also IC?.32 (GPIO21); no longer IC?.14 (GPIO11)
- net SCL_PWR: now also IC?.7 (GPIO5)
- net SDA: now also IC?.9 (RC1)
- net SDA_I2C_1: now also IC?.31 (GPIO20); no longer IC?.13 (GPIO10)
- net SDA_I2C_2: now also IC?.34 (GPIO22); no longer IC?.15 (GPIO12)
- net SDA_PWR: now also IC?.6 (GPIO4)
- net VBATT: now also IC?.2 (GPIO0); no longer IC?.6 (GPIO4)
- net VBATT_SENSE: now also IC?.5 (GPIO3)
- net VBUS_IN: now also IC?.3 (GPIO1)
- net VBUS_RESET: now also IC?.8 (GPIO6)
- net WDT_WDI: no longer IC?.29 (GPIO18)
- net A0: now reaches IC?.38 (GPIO26/ADC0)
- net A0: now also U?.1 (A0)
- net A1: now reaches IC?.39 (GPIO27/ADC1)
- net A1: now also U?.2 (A1)
- net V_SOLAR: no longer names the net of IC?.16 (GPIO13)
- new net: C?.1, C?.1, C?.1, D?.2 (A), L?.1, R?.2, U?.1 (S), U?.2 (S), U?.3 (S)
- new net: C?.2, C?.2, C?.2, L?.1, U?.5 (D), U?.6 (D), U?.7 (D), U?.8 (D)
- new net: C?.2, R?.2, U?.6 (AIN3)
- new net: C?.1, IC?.1 (VOUTA), R?.1, R?.2
- new net: C?.2, IC?.2 (VINA-), R?.1, R?.2
- new net: J?.1 (Pin_1), R?.2, R?.2, R?.2
- new net: C.1, IC?.6 (VCC), R?.2
- new net: C?.1, IC?.6 (VINB-), R?.1, R?.1
- new net: J?.1 (Pin_1), SW?.4 (A)
- new net: C?.1, R?.1, R?.2 (x2)
- new net: C?.1, IC?.3 (VINA+), R?.1
- new net: C?.2, IC?.1 (IN+), R?.2
- new net: C?.1, R?.2, U?.7 (AIN2)
- new net: D?.1 (K), R?.1
- new net: R?.1, R?.2, TH?.1
- new net: C?.2, IC?.7 (VOUTB), R?.1, R?.2
- new net: C?.1, IC?.3 (IN-), R?.1
- new net: R?.1, SW?.1 (A), U?.16 (SCL)
- new net: R?.2, SW?.1 (A), U?.15 (SDA)
- new net: J?.2 (Pin_2), R?.1, R?.1, R?.2
- new net: C?.1, R?.2, U?.10 (AIN1)
- new net: C?.2, IC?.8 (VDD)
- new net: C?.2, U?.4 (G)
- new net: C?.1, IC?.2 (BOOT)
- new net: C?.2, IC?.8 (PHASE)
- new net: IC?.4 (OUT), R?.1
- new net: R?.1, SW?.1 (A), U?.14 (DRDY_N)
- new net: IC?.5 (LOWDR), U?.4 (G)
- new net: C?.1, IC?.1 (HIGHDR)
- new net: D?.2 (A), R?.2
- new net +1V5: R?.1
- new net +8V: C?.1, C?.1, C?.1, C?.1, C?.1, C?.1, C?.1, C?.1, C?.1, C?.1, C?.1, IC?.1 (VIN), J?.2 (Pin_2), R?.1, U?.5 (D), U?.6 (D), U?.7 (D), U?.8 (D)
- new net AMP_VDD: C?.1, IC?.6 (RC4)
- new net BUT: IC?.4 (~{MCLR}/VPP/RA3), J?.1 (Pin_1), SW?.2
- new net DIV_GND: C?.2, C?.2, IC?.2 (RA5), R?.2, R?.2
- new net GNDA: C?.1, C?.1, C?.2, C?.2, C?.2, C?.2, C?.2, IC?.2 (GND), R?.1, R?.1, SW?.2 (B), SW?.2 (B), SW?.2 (B), TH?.2, U?.11 (AIN0), U?.3 (RESET_N), U?.4 (DGND), U?.5 (AGND), U?.8 (REFN)
- new net ISENSE_IN: IC?.8 (RC2), R?.2
- new net LED: IC?.5 (RC5), R?.1
- new net NC0: IC?.3 (PWM), IC?.3 (RA4)
- new net PGC/ISENSE_OUT: IC?.12 (RA1/ICSPCLK), J?.5 (Pin_5), R?.1
- new net PGD_FAULT: IC?.13 (RA0/ICSPDAT), J?.4 (Pin_4)
- new net VSENSE_IN: IC?.11 (RA2)
- new net VSENSE_OUT: IC?.7 (RC3)
- no-connect marks 97 -> 93
Other:
- note added: "5V Regulator (switching)"
- note added: "ADC CONVERTOR"
- note added: "Dual Op-Amps"
- note added: "Fuel Gauge & Cell Balancing connections [don't know if to include?]"
- note added: "LDO"
- note added: "LDO Vltg Reg"
- note added: "MOSFET Driver (5V Buck)"
- note added: "MPPT (AN1521 based)"
- note added: "Microcontroller"
- note removed: "(USB Charging for Battery)"
- note removed: "2S Li-Ion Battery Solar Charging Circuit"
- note removed: "5V Regulator (linear)"
- note removed: "Power Management"
- moved on the sheet: C?
