File: Saddle Board/SpresensePart2.kicad_pcb (KiCad board)
At the start: 2 copper layers, 89.7 x 76.1 mm, 28 parts, among them J1 5040500591, J10 455-1750-1-ND, J11 CONN_01, J12 CONN_01, J15 CONN_01, J16 CONN_01, J2 5040500591, J3 5040500591, J4 5040500591, J5 5040500591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

Commit message: Final As Ordered Feb 1, 2023
Parts:
- added G***: LOGO, LOGO, F.Cu at (113.7, 123.6)
- added G***: LOGO, LOGO, F.Cu at (130.7, 126.9)
Routing:
- net /PA22: track 46.3 -> 45.5 mm
Other:
- board size 89.7 x 76.1 mm -> 89.6 x 59.3 mm
- board text added: "Saddle Board V ? Antony Makar | Nicole Maggard"
